Commit message: Add dual GNSS antenna setting

File: GLIM_plusplus/config/sensor_dome.urdf (robot description, URDF)
Before this commit: robot sensor_dome, 8 links, 7 joints
Links:
- added link gnss_antenna_primary_link
- added link gnss_antenna_secondary_link
Joints:
- added joint imu_to_gnss_antenna_primary_link: type fixed, parent imu_link, child gnss_antenna_primary_link, origin xyz=0.000000 0.000000 0.300000 rpy=0.000000 0.000000 0.000000
- added joint imu_to_gnss_antenna_secondary_link: type fixed, parent imu_link, child gnss_antenna_secondary_link, origin xyz=0.000000 0.000000 0.000000 rpy=0.000000 0.000000 0.000000

Commit message: Add base_link tf as the goal for GICP

File: GLIM_plusplus/config/sensor_dome.urdf (robot description, URDF)
Before this commit: robot sensor_dome, 10 links, 9 joints
Links:
- added link base_link
Joints:
- added joint imu_to_base_link: type fixed, parent imu_link, child base_link, origin xyz=0.000000 0.000000 0.000000 rpy=0.000000 0.000000 0.000000
