Commit message: cherry pick glim++ and gicp++

File: GLIM_plusplus/config/sensor_dome.urdf (robot description, URDF)
Before this commit: robot sensor_dome, 11 links, 10 joints
Links:
- added link cam_front_left_optical_frame
- added link cam_front_right_optical_frame
- added link cam_rear_left_optical_frame
- added link cam_rear_right_optical_frame
Joints:
- removed joint imu_to_base_link
- removed joint imu_to_cam_front_left_link
- removed joint imu_to_cam_front_right_link
- removed joint imu_to_cam_rear_left_link
- removed joint imu_to_cam_rear_right_link
- removed joint imu_to_gnss_antenna_primary_link
- removed joint imu_to_gnss_antenna_secondary_link
- removed joint imu_to_lidar_front_link
- removed joint imu_to_lidar_rear_left_link
- removed joint imu_to_lidar_rear_right_link
- added joint cam_front_left_link_to_cam_front_left_optical_frame: type fixed, parent cam_front_left_link, child cam_front_left_optical_frame, origin xyz=0.000000 0.000000 0.000000 rpy=-1.570796 0.000000 -1.570796
- added joint cam_front_right_link_to_cam_front_right_optical_frame: type fixed, parent cam_front_right_link, child cam_front_right_optical_frame, origin xyz=0.000000 0.000000 0.000000 rpy=-1.570796 0.000000 -1.570796
- added joint cam_rear_left_link_to_cam_rear_left_optical_frame: type fixed, parent cam_rear_left_link, child cam_rear_left_optical_frame, origin xyz=0.000000 0.000000 0.000000 rpy=-1.570796 0.000000 -1.570796
- added joint cam_rear_right_link_to_cam_rear_right_optical_frame: type fixed, parent cam_rear_right_link, child cam_rear_right_optical_frame, origin xyz=0.000000 0.000000 0.000000 rpy=-1.570796 0.000000 -1.570796
- added joint imu_link_to_base_link: type fixed, parent imu_link, child base_link, origin xyz=0.000000 0.000000 0.000000 rpy=0.000000 0.000000 0.000000
- added joint imu_link_to_cam_front_left_link: type fixed, parent imu_link, child cam_front_left_link, origin xyz=0.075000 0.055000 0.126500 rpy=0.000000 0.000000 0.000000
- added joint imu_link_to_cam_front_right_link: type fixed, parent imu_link, child cam_front_right_link, origin xyz=0.075000 -0.055000 0.126500 rpy=0.000000 0.000000 0.000000
- added joint imu_link_to_cam_rear_left_link: type fixed, parent imu_link, child cam_rear_left_link, origin xyz=-0.108122 0.047272 0.126500 rpy=0.000000 0.000000 2.094394
- added joint imu_link_to_cam_rear_right_link: type fixed, parent imu_link, child cam_rear_right_link, origin xyz=-0.108122 -0.047272 0.126500 rpy=0.000000 -0.000000 -2.094394
- added joint imu_link_to_gnss_antenna_primary_link: type fixed, parent imu_link, child gnss_antenna_primary_link, origin xyz=0.000000 0.000000 0.273000 rpy=0.000000 0.000000 0.000000
- added joint imu_link_to_gnss_antenna_secondary_link: type fixed, parent imu_link, child gnss_antenna_secondary_link, origin xyz=0.000000 0.000000 0.000000 rpy=0.000000 0.000000 0.000000
- added joint imu_link_to_lidar_front_link: type fixed, parent imu_link, child lidar_front_link, origin xyz=0.080000 0.000000 0.114500 rpy=0.000000 0.000000 0.000000
- added joint imu_link_to_lidar_rear_left_link: type fixed, parent imu_link, child lidar_rear_left_link, origin xyz=-0.040000 0.069282 0.114500 rpy=0.000000 0.000000 2.094394
- added joint imu_link_to_lidar_rear_right_link: type fixed, parent imu_link, child lidar_rear_right_link, origin xyz=-0.040000 -0.069282 0.114500 rpy=0.000000 -0.000000 -2.094394
